Commit message: update actuator control, added new package to display urdf model and tf tree

File: model/Oxpa-Series/Oxpa/oxpa.urdf (robot description, URDF)
Before this commit: robot oxpa, 10 links, 9 joints
Links:
- removed link camera_front_link
- removed link gripper_left_link
- removed link gripper_right_link
- added link actuator_0_link; visual mesh filename=./oxpa_meshes/dae/actuator_0.dae scale=1.00000 1.00000 1.00000
- added link actuator_1_link; visual mesh filename=./oxpa_meshes/dae/actuator_1.dae scale=1.00000 1.00000 1.00000
- added link oak_d_base_frame; visual mesh filename=./oxpa_meshes/dae/oak-d-lite.dae scale=1.00000 1.00000 1.00000
- added link oak_d_imu_frame
- added link oak_d_left_frame
- added link oak_d_rgb_frame
- added link oak_d_right_frame
- link base_link: mass 1.66000 -> 1.86000
- link rotor_0_link: geometry collision cylinder length=0.006 radius=0.127; visual mesh filename=./oxpa_meshes/dae/rotor0.dae scale=1.00000 1.00000 1.00000
- link rotor_1_link: geometry collision cylinder length=0.006 radius=0.127; visual mesh filename=./oxpa_meshes/dae/rotor1.dae scale=1.00000 1.00000 1.00000
- link rotor_2_link: geometry collision cylinder length=0.006 radius=0.127; visual mesh filename=./oxpa_meshes/dae/rotor2.dae scale=1.00000 1.00000 1.00000
- link rotor_3_link: geometry collision cylinder length=0.006 radius=0.127; visual mesh filename=./oxpa_meshes/dae/rotor3.dae scale=1.00000 1.00000 1.00000
Joints:
- removed joint camera_front_joint
- removed joint gripper_left_joint
- removed joint gripper_right_joint
- removed joint rotor_0
- removed joint rotor_1
- removed joint rotor_2
- removed joint rotor_3
- added joint actuator_0_joint: type revolute, parent base_link, child actuator_0_link, origin xyz=-0.00022 0.02876 -0.09228 rpy=0.00000 0.00000 0.00000, axis 1.00000 0.00000 0.00000, limit lower=-1.57000 upper=1.57000 effort=0.11000 velocity=0.00000
- added joint actuator_1_joint: type revolute, parent base_link, child actuator_1_link, origin xyz=-0.00056 -0.02866 -0.09218 rpy=0.00000 0.00000 0.00000, axis 1.00000 0.00000 0.00000, limit lower=-1.57000 upper=1.57000 effort=0.11000 velocity=0.00000
- added joint oak_d_base_joint: type fixed, parent base_link, child oak_d_base_frame, origin xyz=0.09562 0.00003 -0.04740 rpy=0.00000 0.00000 0.00000
- added joint oak_d_imu_joint: type fixed, parent oak_d_base_frame, child oak_d_imu_frame, origin xyz=-0.00596 -0.03738 0.00323 rpy=0.00000 0.00000 0.00000
- added joint oak_d_left_joint: type fixed, parent oak_d_base_frame, child oak_d_left_frame, origin xyz=-0.00000 0.03753 0.00000 rpy=0.00000 0.00000 0.00000
- added joint oak_d_rgb_joint: type fixed, parent oak_d_base_frame, child oak_d_rgb_frame, origin xyz=0.00000 0.00000 0.00000 rpy=0.00000 0.00000 0.00000
- added joint oak_d_right_joint: type fixed, parent oak_d_base_frame, child oak_d_right_frame, origin xyz=0.00000 -0.03747 0.00000 rpy=0.00000 0.00000 0.00000
- added joint rotor_0_joint: type revolute, parent base_link, child rotor_0_link, origin xyz=0.17281 -0.17000 0.04217 rpy=0.00000 0.00000 0.00000, axis 0.00000 0.00000 1.00000, limit lower=-3.14000 upper=3.14000 effort=0.00000 velocity=0.00000
- added joint rotor_1_joint: type revolute, parent base_link, child rotor_1_link, origin xyz=-0.16699 0.17000 0.04217 rpy=0.00000 0.00000 0.00000, axis 0.00000 0.00000 1.00000, limit lower=-3.14000 upper=3.14000 effort=0.00000 velocity=0.00000
- added joint rotor_2_joint: type revolute, parent base_link, child rotor_2_link, origin xyz=0.17301 0.17000 0.04217 rpy=0.00000 0.00000 0.00000, axis 0.00000 0.00000 1.00000, limit lower=-3.14000 upper=3.14000 effort=0.00000 velocity=0.00000
- added joint rotor_3_joint: type revolute, parent base_link, child rotor_3_link, origin xyz=-0.16699 -0.17000 0.04217 rpy=0.00000 0.00000 0.00000, axis 0.00000 0.00000 1.00000, limit lower=-3.14000 upper=3.14000 effort=0.00000 velocity=0.00000
